Commit message: add realsense

File: turtlebot3_description/urdf/turtlebot3_waffle_pi.urdf.xacro (robot description, xacro)
@@ -3,4 +3,6 @@
   <xacro:include filename="$(find turtlebot3_description)/urdf/common_properties.xacro"/>
   <xacro:include filename="$(find turtlebot3_description)/urdf/turtlebot3_waffle_pi.gazebo.xacro"/>
+  <!-- realsense -->
+  <xacro:include filename="$(find realsense2_description)/urdf/_d435.urdf.xacro" />
   <link name="base_footprint"/>
   <joint name="base_joint" type="fixed">
@@ -185,3 +187,7 @@
   </joint>
   <link name="camera_rgb_optical_frame"/>
+  <!-- realsense -->
+  <xacro:sensor_d435 name="d435" topics_ns="d435" parent="base_link" publish_pointcloud="true">
+    <origin xyz="-0.052 0 0.2" rpy="0 0 0" />
+  </xacro:sensor_d435>
 </robot>
